File: pcb_layout/PCB/LMP2011basedV2.brd (EAGLE design)
At the start: 53.4 x 25.4 mm, 44 parts, among them J1 10118194-0001LF, U1 LMP2011MF, U2 TS5A23167DCUR, U3 TS5A23166DCUR, U4 TS5A23166DCUR, U5 LTC6241CS8PBF, U6 LTC6240CS8PBF, X1 PN87520-S

Commit message: spice models, scripts and pcb layouts update
Parts:
- removed C6: 10p, resistor:C0805
- added C2: 10p, resistor:C0805
- R1: value 10k -> 1k
- R10: value 1k -> 100k
- R11: value 100k -> 1k
- R12: value 10k -> 1M
- R13: value 1M -> 10k
- R17: value 10k -> 1K@1MHz
- R18: value 1K@1MHz -> 10k
- R20: value 10k -> 100k
- R21: value 49.9 -> 10k; device resistor:R0603 -> resistor:R0805
- R26: value 100k -> 49.9; device resistor:R0805 -> resistor:R0603
- U1: value LMP2011MF -> TS5A23167DCUR; device LMP2011MF:SOT95P285X120-5N -> TS5A2316XDCUR:SOP50P310X90-8N
- U2: value TS5A23167DCUR -> LMP2011MF; device TS5A2316XDCUR:SOP50P310X90-8N -> LMP2011MF:SOT95P285X120-5N
- moved R26 54.9 mm to (14.6, 14.3), flipped to the bottom
- moved R20 37.7 mm to (-2.86, -12.4), flipped to the top, turned to 0 degrees
- moved C5 34.0 mm to (34.3, 18.4), flipped to the bottom, turned to 0 degrees
- moved R17 33.9 mm to (47.9, 23.8), flipped to the top, turned to 0 degrees
- moved R18 33.9 mm to (14.6, 17.8), flipped to the bottom, turned to 180 degrees
- moved C3 13.6 mm to (13.0, 7.62), turned to 180 degrees
- moved C4 11.1 mm to (1.91, 7.94), turned to 90 degrees
- moved U1 10.5 mm to (29.8, 4.45), flipped to the bottom, turned to 90 degrees
- moved U2 10.5 mm to (29.5, 14.9), flipped to the top, turned to 0 degrees
- moved R21 9.53 mm to (24.1, 14.0), turned to 90 degrees
- moved R22 6.35 mm to (-2.86, -18.7)
- moved R24 6.35 mm to (-2.86, -31.4)
- moved R23 6.35 mm to (-2.86, -25.1)
- moved R25 6.35 mm to (-2.86, -37.8)
Connections:
- net +5V: now also R17.1, U1.8, U2.5; no longer R18.1, U1.5, U2.8
- net +5V_USB: now also R17.2; no longer R18.2
- net ADC__VOLT: now also R26.2; no longer R21.2
- net GND: now also R18.1, R20.1, U1.4, U2.2; no longer R17.1, R26.1, U1.2, U2.4
- net N$1: now also R18.2; no longer R17.2
- net N$10: now also C2.2, U2.4; no longer C3.2, U1.4
- net N$11: now also C4.1; no longer C5.1
- net N$12: now also U2.3; no longer U1.3
- net N$13: now also C3.2; no longer C4.2
- net N$15: now also C4.2; no longer C5.2
- net N$2: now also C5.1, R21.2, R26.1; no longer C6.1, R20.2, R21.1
- net N$4: now also C5.2, R21.1; no longer C6.2, R20.1
- net N$7: now also C3.1; no longer C4.1
- net OUT_STAGE1: now also C2.1, U2.1; no longer C3.1, U1.1
- net SWITCH_CTRL_1: now also R20.2, U1.3, U1.7; no longer R22.2, U2.3, U2.7
- net SWITCH_CTRL_2: now also R22.2; no longer R23.2
- net SWITCH_CTRL_3: now also R23.2; no longer R24.2
- net SWITCH_CTRL_4: now also R24.2; no longer R25.2
- net SWITCH_CTRL_5: now also R25.2; no longer R26.2
- net VMCU: now also U1.1, U1.5; no longer U2.1, U2.5
- net VS-: now also U1.2, U1.6; no longer U2.2, U2.6
