File: pcb_layout/PCB/LMP2011basedV2.sch (EAGLE design)
At the start: 44 parts, among them J1 10118194-0001LF, U1 LMP2011MF, U2 TS5A23167DCUR, U3 TS5A23166DCUR, U4 TS5A23166DCUR, U5 LTC6241CS8PBF, U6 LTC6240CS8PBF, X1 PN87520-S

Commit message: spice models, scripts and pcb layouts update
Parts:
- removed C6: 10p, resistor:C-EUC0805
- added C2: 10p, resistor:C-EUC0805
- R1: value 10k -> 1k
- R10: value 1k -> 100k
- R11: value 100k -> 1k
- R12: value 10k -> 1M
- R13: value 1M -> 10k
- R17: value 10k -> 1K@1MHz
- R18: value 1K@1MHz -> 10k
- R20: value 10k -> 100k
- R21: value 49.9 -> 10k; device resistor:R-US_R0603 -> resistor:R-US_R0805
- R26: value 100k -> 49.9; device resistor:R-US_R0805 -> resistor:R-US_R0603
- U1: value LMP2011MF -> TS5A23167DCUR; device LMP2011MF:LMP2011MF -> TS5A2316XDCUR:TS5A23167DCUR
- U2: value TS5A23167DCUR -> LMP2011MF; device TS5A2316XDCUR:TS5A23167DCUR -> LMP2011MF:LMP2011MF
Connections:
- net +5V: now also R17.1; no longer R18.1
- net +5V_USB: now also R17.2; no longer R18.2
- net ADC__VOLT: now also R26.2; no longer R21.2
- net GND: now also R18.1, R20.1, U1.GND, U2.V-; no longer R17.1, R26.1, U1.V-, U2.GND
- net N$1: now also R18.2; no longer R17.2
- net N$10: now also C2.2, U2.VIN-; no longer C3.2, U1.VIN-
- net N$11: now also C4.1; no longer C5.1
- net N$12: now also U2.VIN+; no longer U1.VIN+
- net N$13: now also C3.2; no longer C4.2
- net N$15: now also C4.2; no longer C5.2
- net N$2: now also C5.1, R21.2, R26.1; no longer C6.1, R20.2, R21.1
- net N$4: now also C5.2, R21.1; no longer C6.2, R20.1
- net N$7: now also C3.1; no longer C4.1
- net OUT_STAGE1: now also C2.1, U2.VOUT; no longer C3.1, U1.VOUT
- net SWITCH_CTRL_1: now also R20.2, U1.IN1, U1.IN2; no longer R22.2, U2.IN1, U2.IN2
- net SWITCH_CTRL_2: now also R22.2; no longer R23.2
- net SWITCH_CTRL_3: now also R23.2; no longer R24.2
- net SWITCH_CTRL_4: now also R24.2; no longer R25.2
- net SWITCH_CTRL_5: now also R25.2; no longer R26.2
- net VMCU: now also U1.NC1, U1.NC2; no longer U2.NC1, U2.NC2
- net VS-: now also U1.COM1, U1.COM2; no longer U2.COM1, U2.COM2
Other:
- moved on the sheet: C3, C4, C5, R17, R18, R20, R21, R22, R23, R24, R25, R26
