File: pcb_layout/PCB/MAX4239basedV3.brd (EAGLE design)
At the start: 53.3 x 25.4 mm, 45 parts, among them J1 10118194-0001LF, U1 MAX4239ASA, U2 TS5A23167DCUR, U3 TS5A23166DCUR, U4 TS5A23166DCUR, U5 LTC6241CS8PBF, U6 LTC6240CS8PBF, X1 PN87520-S

Commit message: spice models, scripts and pcb layouts update
Parts:
- added C4: 2u, resistor:PANASONIC_B
- added C7: 10u, resistor:PANASONIC_B
- added D3: CUS08F30, CUS08F30:SOD323
- added R26: 1k, resistor:R0805
- added R27: 10uH, resistor:R1210
- added R28: 35k, resistor:R0805
- added R29: 10k, resistor:R0805
- added U7: MIC2250, MIC2250:SOT95P270X145-5N
- C2: value 0.1u -> 1m
- R10: value 1k -> 100K
- R11: value 100k -> 1K
- R12: value 10k -> 1M
- R13: value 1M -> 10K
Connections:
- removed net N$9: C2.-, U1.1
- new net +5V5: C2.+, C4.+, D3.C, R28.2, U1.1, U1.7
- new net FB: R28.1, R29.2, U7.3
- new net SW: D3.A, R27.2, U7.1
- net +5V: now also C7.+, R27.1, U7.4, U7.5; no longer C2.+, U1.7
- net DGND: now also U7.2
- net GND: now also C2.-, C4.-, C7.-, R26.1, R29.1
- net OUT_STAGE1: now also R26.2
Routing:
- net N$9: track 26.6 -> 0.00 mm
- net +5V: track 77.5 -> 73.8 mm
