File: pcb_layout/PCB/MAX4239/MAX4239basedV3.brd (EAGLE design)
At the start: 53.3 x 25.4 mm, 53 parts, among them J1 10118194-0001LF, U1 MAX4239ASA, U2 TS5A23167DCUR, U3 TS5A23166DCUR, U4 TS5A23166DCUR, U5 LTC6241CS8PBF, U6 LTC6240CS8PBF, U7 MIC2250, X1 PN87520-S

Commit message: Added stage images for MAX4239 circuit and README
	nuevo archivo: pcb_layout/PCB/LMP2011/README.md
	nuevo archivo: pcb_layout/PCB/MAX4239/Images/IM1.png
	nuevo archivo: pcb_layout/PCB/MAX4239/Images/IM2.png
	nuevo archivo: pcb_layout/PCB/MAX4239/Images/IM3.png
	nuevo archivo: pcb_layout/PCB/MAX4239/Images/IM4.png
	nuevo archivo: pcb_layout/PCB/MAX4239/Images/IM5.png
	nuevo archivo: pcb_layout/PCB/MAX4239/Images/IM6.png
	nuevo archivo: pcb_layout/PCB/MAX4239/Images/IM7.png
	modificado:    pcb_layout/PCB/MAX4239/MAX4239basedV3.brd
	modificado:    pcb_layout/PCB/MAX4239/MAX4239basedV3.sch
	nuevo archivo: pcb_layout/PCB/MAX4239/README.md
Parts:
- R1, R2: value 10k -> 1k
Changed lines of the file:
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@@
 <attribute name="VALUE" x="46.99" y="20.6375" size="1.27" layer="27"/>
 </element>
-<element name="R1" library="resistor" library_urn="urn:adsk.eagle:library:348" package="R0805" package3d_urn="urn:adsk.eagle:package:26059/1" value="10k" x="37.465" y="10.795" smashed="yes">
+<element name="R1" library="resistor" library_urn="urn:adsk.eagle:library:348" package="R0805" package3d_urn="urn:adsk.eagle:package:26059/1" value="1k" x="37.465" y="10.795" smashed="yes">
 <attribute name="NAME" x="37.465" y="12.065" size="0.8128" layer="25"/>
 <attribute name="VALUE" x="36.83" y="8.255" size="1.27" layer="27"/>
@@
 <attribute name="VALUE" x="34.925" y="17.145" size="1.27" layer="28" rot="MR270"/>
 </element>
-<element name="R2" library="resistor" library_urn="urn:adsk.eagle:library:348" package="R0805" package3d_urn="urn:adsk.eagle:package:26059/1" value="10k" x="26.9875" y="1.905" smashed="yes">
+<element name="R2" library="resistor" library_urn="urn:adsk.eagle:library:348" package="R0805" package3d_urn="urn:adsk.eagle:package:26059/1" value="1k" x="26.9875" y="1.905" smashed="yes">
 <attribute name="NAME" x="25.4" y="3.175" size="0.8128" layer="25"/>
 <attribute name="VALUE" x="26.3525" y="-0.635" size="1.27" layer="27"/>
