File: pcb_layout/PCB/MAX4239/MAX4239basedV3.sch (EAGLE design)
At the start: 53 parts, among them J1 10118194-0001LF, U1 MAX4239ASA, U2 TS5A23167DCUR, U3 TS5A23166DCUR, U4 TS5A23166DCUR, U5 LTC6241CS8PBF, U6 LTC6240CS8PBF, U7 MIC2250, X1 PN87520-S

Commit message: Added stage images for MAX4239 circuit and README
	nuevo archivo: pcb_layout/PCB/LMP2011/README.md
	nuevo archivo: pcb_layout/PCB/MAX4239/Images/IM1.png
	nuevo archivo: pcb_layout/PCB/MAX4239/Images/IM2.png
	nuevo archivo: pcb_layout/PCB/MAX4239/Images/IM3.png
	nuevo archivo: pcb_layout/PCB/MAX4239/Images/IM4.png
	nuevo archivo: pcb_layout/PCB/MAX4239/Images/IM5.png
	nuevo archivo: pcb_layout/PCB/MAX4239/Images/IM6.png
	nuevo archivo: pcb_layout/PCB/MAX4239/Images/IM7.png
	modificado:    pcb_layout/PCB/MAX4239/MAX4239basedV3.brd
	modificado:    pcb_layout/PCB/MAX4239/MAX4239basedV3.sch
	nuevo archivo: pcb_layout/PCB/MAX4239/README.md
Parts:
- R1, R2: value 10k -> 1k
Other:
- note added: "5V5"
- note removed: "+8V68 SUPPLY"
- moved on the sheet: C2, C3, C5, C6, D1, D2, J1, JP1, JP2, JP4, L1, R1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
