File: pcb_layout/PCB/LMP2011/LMP2011basedV2.sch (EAGLE design)
At the start: 44 parts, among them J1 10118194-0001LF, U1 TS5A23167DCUR, U2 LMP2011MF, U3 TS5A23166DCUR, U4 TS5A23166DCUR, U5 LTC6241CS8PBF, U6 LTC6240CS8PBF, X1 PN87520-S

Commit message: Added figures for LMP2011
Parts:
- added R27: 1k, resistor:R-US_R0805
Connections:
- net GND: now also R27.2
- net OUT_STAGE1: now also R27.1
Other:
- moved on the sheet: C5, D1, D2, J1, JP1, R16, R17, R18, R19, R21, R26, U6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
